File: USB_LEDs_2835.kicad_pcb (KiCad board)
At the start: 2 copper layers, 99.9 x 20 mm, 55 parts, among them U1 MT9284, U2 JL8022W-L, U3 74LVC1G04

Commit message: Add files via upload
Parts:
- moved C1 1.64 mm to (42.9, 44.3)
- moved JP2 1.45 mm to (35.9, 39.2), turned to 90 degrees
- moved U2 0.67 mm to (39.0, 48.2)
- moved R6 0.60 mm to (36.5, 44.5)
- moved JP1 0.15 mm to (39.8, 39.2)
Connections:
- JP2 pad 1: +5V -> GND
- JP2 pad 3: GND -> +5V
Routing:
- net GND: track 124.0 -> 156.2 mm, vias 4 -> 0
- net Net-(JP1-Pad2): track 16.0 -> 11.3 mm
- net +5V: track 200.8 -> 202.3 mm
- net Net-(C5-Pad1): track 4.75 -> 5.90 mm
- net Net-(D33-Pad2): track 95.2 -> 95.8 mm
- net Net-(U2-Pad8): track 17.8 -> 18.4 mm
- removed copper zone on B.Cu, net GND

Commit message: Add files via upload
Routing:
- net GND: track 156.2 -> 158.3 mm
- net Net-(JP1-Pad2): track 11.3 -> 12.1 mm

Commit message: Add files via upload
Parts:
- D1, D10, D11, D12, D13, D14, D15, D16, D17, D18, D19, D2, D20, D21, D22, D23, D24, D25, D26, D27, D28, D29, D3, D30, D31, D32, D4, D5, D6, D7, D8, D9: footprint LED_SMD:LED_2835 -> LED_SMD:LED_2835_custom_margin
- R1: footprint Resistor_SMD:R_0402_1005Metric -> Resistor_SMD:R_0603_1608Metric
- moved R1 1.57 mm to (118.8, 47.3)
- moved R2 1.36 mm to (120.9, 46.2), turned to 0 degrees
- moved C5 0.46 mm to (41.0, 51.8)
Routing:
- net Net-(D16-Pad1): track 93.6 -> 261.6 mm
- net +5V: track 202.3 -> 153.5 mm
- net GND: track 158.3 -> 155.9 mm
- net Net-(R1-Pad2): track 2.92 -> 4.16 mm
