File: USB_LEDs_2835.kicad_sch (KiCad schematic)
At the start: 55 parts, among them U1 MT9284, U2 JL8022W-L, U3 74LVC1G04

Commit message: Add files via upload
Connections:
- net +5V: now also JP2.3 (B); no longer JP2.1 (A)
- net GND: now also JP2.1 (A); no longer JP2.3 (B)
Other:
- moved on the sheet: C2, H1, H2

Commit message: Add files via upload
Parts:
- D1, D10, D11, D12, D13, D14, D15, D16, D17, D18, D19, D2, D20, D21, D22, D23, D24, D25, D26, D27, D28, D29, D3, D30, D31, D32, D4, D5, D6, D7, D8, D9: footprint LED_SMD:LED_2835 -> LED_SMD:LED_2835_custom_margin
- R1: footprint Resistor_SMD:R_0402_1005Metric -> Resistor_SMD:R_0603_1608Metric
