File: USB_LEDs_2835/USB_LEDs_2835.kicad_sch (KiCad schematic)
At the start: 55 parts, among them U1 MT9284, U2 JL8022W-L, U3 74LVC1G04

Commit message: Add files via upload
Parts:
- added D35: TVS, Diode_SMD:D_SOD-923, symbol Device:D_TVS_unidirection
- C2: value 1u -> 22u
- L1: footprint Inductor_SMD:L_0530_custom -> Inductor_SMD:L_WHC_0630_custom
- R1: value 5k -> 23.2k
- R2, R3: value 10k -> 200k
- Rx1: value 100m -> 1.5
- TP1: footprint TestPoint:TestPoint_Loop_D2.50mm_Drill1.0mm -> TestPoint:TestPoint_Loop_D2.50mm_Drill1.0mm_overlap_pad_custom
Connections:
- net +5V: now also D35.2 (A2)
- net GND: now also D35.1 (A1)

Commit message: Add files via upload
Parts:
- removed D35: TVS, Diode_SMD:D_SOD-923, symbol Device:D_TVS_unidirection
- removed U1: MT9284, Package_TO_SOT_SMD:SOT-23-6, symbol USB_LED_Lib:MT9284
- removed U2: JL8022W-L, Package_SO:SOIC-8_3.9x4.9mm_P1.27mm, symbol USB_LED_Lib:JL8022W-L
- removed U3: 74LVC1G04, Package_TO_SOT_SMD:SOT-353_SC-70-5, symbol USB_LED_Lib:74LVC1G04
- added D35: D_TVS_unidirection, Diode_SMD:D_SOD-923, symbol custom_symbol:D_TVS_unidirection
- added U1: MT9284_1, Package_TO_SOT_SMD:SOT-23-6, symbol custom_symbol:MT9284_1
- added U2: JL8022W-L, Package_SO:SOIC-8_3.9x4.9mm_P1.27mm, symbol custom_symbol:JL8022W-L
- added U3: 74LVC1G04, Package_TO_SOT_SMD:SOT-353_SC-70-5, symbol custom_symbol:74LVC1G04
Connections:
- net +5V: now also D35.1 (A1), U1.6 (VIN), U2.3 (VDD), U3.5 (VCC)
- net GND: now also D35.2 (A2), U1.2 (GND), U2.4 (GND), U3.3 (GND)
- net at C5.1: now also U2.2 (VC)
- net at R6.2: now also U2.5 (TI)
- net at JP1.2 (C): now also U2.6 (OPT1)
- net at D33.2 (A): now also U2.7 (SO), U3.2
- net at JP2.2 (C): now also U2.8 (OPT2)
- net at Cx1.1, D1.2 (A), D17.2 (A)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: now also U1.5 (OV)
- net at D34.2 (A), L1.2: now also U1.1 (SW)
- net at R3.1: now also U3.4
- net at R1.2, R2.1: now also U1.3 (FB)
- net at C4.1, D33.1 (K), R4.2: now also U1.4 (EN)
