File: USB_LEDs_2835/USB_LEDs_2835.kicad_sch (KiCad schematic)
At the start: 56 parts, among them U1 MT9284_1, U2 JL8022W-L, U3 74LVC1G04

Commit message: Add files via upload
Parts:
- L1: footprint Inductor_SMD:L_WHC_0630_custom -> custom_footprint_library:L_WHC_0630_custom
- Rx1: footprint Resistor_SMD:R_1206_3216Metric -> custom_footprint_library:R_1206_0805_3216Metric_custom
Changed lines of the file:
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@@
     (property "Reference" "L1" (id 0) (at 129.413 51.435 90))
     (property "Value" "L_Ferrite_Small" (id 1) (at 129.413 53.975 90))
-    (property "Footprint" "Inductor_SMD:L_WHC_0630_custom" (id 2) (at 129.413 56.515 0)
+    (property "Footprint" "custom_footprint_library:L_WHC_0630_custom" (id 2) (at 129.413 56.515 0)
       (effects (font (size 1.27 1.27)) hide)
     )
@@
       (effects (font (size 1.27 1.27)) (justify left))
     )
-    (property "Footprint" "Resistor_SMD:R_1206_3216Metric" (id 2) (at 128.143 86.995 0)
+    (property "Footprint" "custom_footprint_library:R_1206_0805_3216Metric_custom" (id 2) (at 128.143 86.995 0)
       (effects (font (size 1.27 1.27)) hide)
     )
@@
     )
     (path "/43abfdee-8911-49ba-9ef6-3447815c3b58"
-      (reference "L1") (unit 1) (value "L_Ferrite_Small") (footprint "Inductor_SMD:L_WHC_0630_custom")
+      (reference "L1") (unit 1) (value "L_Ferrite_Small") (footprint "custom_footprint_library:L_WHC_0630_custom")
     )
     (path "/46b40edc-42cc-446d-adb2-e52631d88862"
@@
     )
     (path "/98753c78-a4c2-4a80-8ed5-3f6f93aecf71"
-      (reference "Rx1") (unit 1) (value "1.5") (footprint "Resistor_SMD:R_1206_3216Metric")
+      (reference "Rx1") (unit 1) (value "1.5") (footprint "custom_footprint_library:R_1206_0805_3216Metric_custom")
     )
     (path "/437f8d09-8f17-4205-b86b-2fcaa45bda5d"

Commit message: Add files via upload
Parts:
- C2: footprint Capacitor_SMD:C_0402_1005Metric -> Capacitor_SMD:C_0603_1608Metric
Changed lines of the file:
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@@
       (effects (font (size 1.27 1.27)) (justify left))
     )
-    (property "Footprint" "Capacitor_SMD:C_0402_1005Metric" (id 2) (at 180.086 36.576 0)
+    (property "Footprint" "Capacitor_SMD:C_0603_1608Metric" (id 2) (at 180.086 36.576 0)
       (effects (font (size 1.27 1.27)) hide)
     )
@@
     )
     (path "/026f09c8-400d-46f9-844e-0be8161f9746"
-      (reference "C2") (unit 1) (value "22u") (footprint "Capacitor_SMD:C_0402_1005Metric")
+      (reference "C2") (unit 1) (value "22u") (footprint "Capacitor_SMD:C_0603_1608Metric")
     )
     (path "/bc5de113-9719-4067-b963-db31416212e7"
