File: USB_LEDs_2835/USB_LEDs_2835.kicad_pcb (KiCad board)
At the start: 2 copper layers, 99.9 x 20 mm, 53 parts, among them U1 MT9284, U2 JL8022W-L, U3 74LVC1G04

Commit message: Add files via upload
Parts:
- added JP1: solderjumper_1, Jumper:SolderJumper-3_P1.3mm_Bridged12_Pad1.0x1.5mm_NumberLabels, F.Cu at (39.8, 39.2)
- added JP2: solderjumper_2, Jumper:SolderJumper-3_P1.3mm_Bridged12_Pad1.0x1.5mm_NumberLabels, F.Cu at (35.9, 39.2)
- Cx1: value 1u -> 22u; footprint Capacitor_SMD:C_0402_1005Metric -> Capacitor_SMD:C_0603_1608Metric
- D1, D10, D11, D12, D13, D14, D15, D16, D17, D18, D19, D2, D20, D21, D22, D23, D24, D25, D26, D27, D28, D29, D3, D30, D31, D32, D4, D5, D6, D7, D8, D9: footprint LED_SMD:LED_2835 -> LED_SMD:LED_2835_custom_margin
- R1: footprint Resistor_SMD:R_0402_1005Metric -> Resistor_SMD:R_0603_1608Metric
- moved R6 3.54 mm to (36.5, 44.5), turned to -90 degrees
- moved C1 1.64 mm to (42.9, 44.3)
- moved R1 1.57 mm to (118.8, 47.3)
- moved R2 1.37 mm to (120.9, 46.2), turned to 0 degrees
- moved U2 0.67 mm to (39.0, 48.2)
- moved C5 0.46 mm to (41.0, 51.8)
- moved Cx1 0.18 mm to (118.2, 43.9)
Connections:
- U2 pad 6: +5V -> Net-(JP1-Pad2)
- U2 pad 8: GND -> Net-(JP2-Pad2)
Routing:
- net Net-(D16-Pad1): track 93.6 -> 261.6 mm
- net +5V: track 197.8 -> 154.5 mm
- net GND: track 130.0 -> 159.7 mm
- net Net-(JP2-Pad2): track 0.00 -> 18.2 mm
- net Net-(JP1-Pad2): track 0.00 -> 12.1 mm
- net Net-(R1-Pad2): track 2.92 -> 4.15 mm
- net Net-(C5-Pad1): track 4.75 -> 5.64 mm
- net Net-(Cx1-Pad1): track 38.5 -> 39.4 mm
- net Net-(D33-Pad2): track 94.5 -> 95.4 mm
- net Net-(R6-Pad1): track 3.40 -> 2.67 mm
- added copper zone on F.Cu, net unconnected-(U3-Pad1)

Commit message: Add files via upload
Parts:
- D33: footprint Diode_SMD:D_SOD-323 -> Diode_SMD:D_SOD-323_custom
- moved U3 0.67 mm to (121.9, 50.8)
Routing:
- net GND: track 159.7 -> 160.6 mm

Commit message: Add files via upload
Parts:
- moved Cx1 2.71 mm to (118.7, 46.5), turned to -90 degrees
- moved R1 2.28 mm to (118.7, 49.5)
- moved Rx1 1.89 mm to (116.8, 48.9)
- moved D34 1.16 mm to (117.8, 40.6)
- moved R2 1.11 mm to (120.8, 47.3)
- moved R4 1.09 mm to (126.3, 48.9)
- moved C4 1.08 mm to (125.3, 48.9)
- moved C3 1.06 mm to (121.3, 48.8)
- moved R3 1.06 mm to (120.3, 48.9)
- moved C2 1.04 mm to (125.7, 47.2)
- moved C5 0.83 mm to (41.8, 51.5)
- moved U1 0.66 mm to (122.3, 44.3)
- moved D33 0.65 mm to (123.8, 47.8)
- moved JP2 0.52 mm to (36.4, 39.2)
- moved U3 0.47 mm to (121.9, 51.3)
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Routing:
- net Net-(D34-Pad2): track 4.30 -> 8.74 mm
- net +5V: track 154.5 -> 150.7 mm
- net GND: track 160.6 -> 158.7 mm
- net Net-(D16-Pad1): track 261.6 -> 259.8 mm
- net Net-(Cx1-Pad1): track 39.4 -> 41.3 mm
- net Net-(JP2-Pad2): track 18.2 -> 17.1 mm
- net Net-(R1-Pad2): track 4.15 -> 5.19 mm
- net Net-(C5-Pad1): track 5.64 -> 4.90 mm
- net Net-(R3-Pad1): track 2.10 -> 1.53 mm
- net Net-(D33-Pad2): track 94.9 -> 94.3 mm

Commit message: Add files via upload
Routing:
- net GND: track 158.7 -> 158.2 mm
Changed lines of the file:
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@@
     (property "Sheetname" "")
     (attr smd)
-    (fp_text reference "D34" (at 0.84 -2.11 90) (layer "F.SilkS")
+    (fp_text reference "D34" (at 3.93 0.02 180) (layer "F.SilkS")
       (effects (font (size 0.5 0.5) (thickness 0.1)))
     )
@@
     (property "Sheetname" "")
     (attr smd)
-    (fp_text reference "Cx1" (at -1.715 0) (layer "F.SilkS")
+    (fp_text reference "Cx1" (at -0.775 0.995 90) (layer "F.SilkS")
       (effects (font (size 0.3 0.3) (thickness 0.07)))
     )
@@
   (segment (start 125.28 48.375) (end 125.275 48.38) (width 0.3) (layer "F.Cu") (net 1))
   (segment (start 123.775 45.5375) (end 123.4475 45.21) (width 0.3) (layer "F.Cu") (net 1))
+  (segment (start 118.675 47.3) (end 116.8975 47.3) (width 0.3) (layer "F.Cu") (net 2))
   (segment (start 125.275 49.34) (end 126.265 49.34) (width 0.3) (layer "F.Cu") (net 2))
   (segment (start 122.25 48.35) (end 122.25 48.05) (width 0.3) (layer "F.Cu") (net 2))
-  (segment (start 127.125 47.175) (end 126.21 47.175) (width 0.3) (layer "F.Cu") (net 2))
   (segment (start 121.1725 44.26) (end 122.03 44.26) (width 0.3) (layer "F.Cu") (net 2))
-  (segment (start 119.81 46.53) (end 119.81 44.26) (width 0.3) (layer "F.Cu") (net 2))
   (segment (start 37.975 48.25) (end 35.3 48.25) (width 0.2) (layer "F.Cu") (net 2))
   (segment (start 122.39 48.21) (end 124.15 48.21) (width 0.3) (layer "F.Cu") (net 2))
-  (segment (start 118.5375 47.4375) (end 118.675 47.3) (width 0.3) (layer "F.Cu") (net 2))
+  (segment (start 116.8975 47.3) (end 116.76 47.4375) (width 0.3) (layer "F.Cu") (net 2))
   (segment (start 122.25 49.3) (end 122.25 48.35) (width 0.3) (layer "F.Cu") (net 2))
   (segment (start 124.55 49.34) (end 125.275 49.34) (width 0.3) (layer "F.Cu") (net 2))
   (segment (start 41.95 45.03) (end 41.95 40.55) (width 0.25) (layer "F.Cu") (net 2))
+  (segment (start 121.1725 44.26) (end 120.18 44.26) (width 0.3) (layer "F.Cu") (net 2))
   (segment (start 35.3 48.25) (end 35.2 48.35) (width 0.2) (layer "F.Cu") (net 2))
   (segment (start 41.32 53.1) (end 122.892772 53.1) (width 0.3) (layer "F.Cu") (net 2))
   (segment (start 122.25 44.48) (end 122.25 48.05) (width 0.3) (layer "F.Cu") (net 2))
-  (segment (start 118.675 47.3) (end 119.04 47.3) (width 0.3) (layer "F.Cu") (net 2))
   (segment (start 41.475 46.345) (end 40.33 46.345) (width 0.25) (layer "F.Cu") (net 2))
-  (segment (start 119.81 44.26) (end 121.1725 44.26) (width 0.3) (layer "F.Cu") (net 2))
   (segment (start 35.2 48.35) (end 35.2 49.43548) (width 0.2) (layer "F.Cu") (net 2))
-  (segment (start 126.32 49.395) (end 127.125 49.395) (width 0.3) (layer "F.Cu") (net 2))
   (segment (start 124.54 48.6) (end 124.54 49.33) (width 0.3) (layer "F.Cu") (net 2))
   (segment (start 35.2 49.43548) (end 35.28452 49.52) (width 0.2) (layer "F.Cu") (net 2))
+  (segment (start 119.59 46.61) (end 118.9 47.3) (width 0.3) (layer "F.Cu") (net 2))
   (segment (start 41.95 45.03) (end 42.975 45.03) (width 0.25) (layer "F.Cu") (net 2))
+  (segment (start 120.18 44.26) (end 119.59 44.85) (width 0.3) (layer "F.Cu") (net 2))
   (segment (start 35.28452 49.52) (end 38.14 49.52) (width 0.2) (layer "F.Cu") (net 2))
   (segment (start 36.496015 51.525) (end 38.1 51.525) (width 0.3) (layer "F.Cu") (net 2))
@@
   (segment (start 38.425 48.25) (end 37.975 48.25) (width 0.25) (layer "F.Cu") (net 2))
   (segment (start 41.475 46.345) (end 42.975 46.345) (width 0.25) (layer "F.Cu") (net 2))
+  (segment (start 127.02 47.175) (end 126.21 47.175) (width 0.3) (layer "F.Cu") (net 2))
   (segment (start 122.25 48.35) (end 122.39 48.21) (width 0.3) (layer "F.Cu") (net 2))
   (segment (start 125.275 51.163249) (end 125.275 49.34) (width 0.3) (layer "F.Cu") (net 2))
+  (segment (start 126.32 49.395) (end 127.02 49.395) (width 0.3) (layer "F.Cu") (net 2))
   (segment (start 122.25 49.3) (end 122.25 49.359879) (width 0.3) (layer "F.Cu") (net 2))
   (segment (start 121.75 50.66) (end 122.78 50.66) (width 0.3) (layer "F.Cu") (net 2))
   (segment (start 31.975 42.45) (end 31.975 44.352335) (width 0.3) (layer "F.Cu") (net 2))
+  (segment (start 118.9 47.3) (end 118.675 47.3) (width 0.3) (layer "F.Cu") (net 2))
   (segment (start 121.96 50.06) (end 121.886569 50.133431) (width 0.3) (layer "F.Cu") (net 2))
   (segment (start 121.32 49.3) (end 122.25 49.3) (width 0.3) (layer "F.Cu") (net 2))
-  (segment (start 119.04 47.3) (end 119.81 46.53) (width 0.3) (layer "F.Cu") (net 2))
   (segment (start 124.54 49.33) (end 124.55 49.34) (width 0.3) (layer "F.Cu") (net 2))
+  (segment (start 119.59 44.85) (end 119.59 46.61) (width 0.3) (layer "F.Cu") (net 2))
   (segment (start 41.32 51.525) (end 41.32 53.1) (width 0.3) (layer "F.Cu") (net 2))
   (segment (start 38.14 49.52) (end 38.14 51.428432) (width 0.2) (layer "F.Cu") (net 2))
-  (segment (start 116.76 47.4375) (end 118.5375 47.4375) (width 0.3) (layer "F.Cu") (net 2))
   (segment (start 122.03 44.26) (end 122.25 44.48) (width 0.3) (layer "F.Cu") (net 2))
   (segment (start 40.33 46.345) (end 38.425 48.25) (width 0.25) (layer "F.Cu") (net 2))
@@
   (segment (start 121.31 49.31) (end 121.32 49.3) (width 0.3) (layer "F.Cu") (net 2))
   (segment (start 41.95 40.55) (end 39.75 40.55) (width 0.25) (layer "F.Cu") (net 2))
-  (segment (start 127.125 49.395) (end 127.125 47.175) (width 0.3) (layer "F.Cu") (net 2))
+  (segment (start 127.02 49.395) (end 127.02 47.175) (width 0.3) (layer "F.Cu") (net 2))
   (segment (start 121.75 50.19) (end 121.75 50.66) (width 0.3) (layer "F.Cu") (net 2))
   (arc (start 122.892772 53.1) (mid 123.924956 52.894685) (end 124.8 52.31) (width 0.3) (layer "F.Cu") (net 2))

Commit message: Add files via upload
Parts:
- added D35: TVS, Diode_SMD:D_SOD-923, F.Cu at (129.5, 43.7)
- C2: value 1u -> 22u
- L1: footprint Inductor_SMD:L_0530_custom -> Inductor_SMD:L_WHC_0630_custom
- R1: value 5k -> 23.2k
- R2, R3: value 10k -> 200k
- Rx1: value 100m -> 1.5
- TP1: footprint TestPoint:TestPoint_Loop_D2.50mm_Drill1.0mm -> TestPoint:TestPoint_Loop_D2.50mm_Drill1.0mm_overlap_pad_custom
- moved R4 4.82 mm to (121.7, 47.6), turned to 0 degrees
- moved C4 4.27 mm to (121.7, 46.6), turned to 180 degrees
- moved C2 3.74 mm to (123.7, 44.0), turned to -90 degrees
- moved C3 1.95 mm to (119.5, 48.0)
- moved R2 1.86 mm to (119.1, 46.6)
- moved R3 1.85 mm to (118.6, 48.0)
- moved JP1 1.76 mm to (41.0, 38.0)
- moved JP2 1.76 mm to (37.6, 38.0)
- moved Cx1 1.69 mm to (117.6, 45.2), turned to 0 degrees
- moved U3 1.29 mm to (121.6, 50.0)
- moved D33 1.25 mm to (124.2, 46.6)
- moved R1 1.16 mm to (118.8, 50.7)
- moved U1 1.11 mm to (121.2, 44.4)
- moved R6 0.55 mm to (36.6, 45.0), turned to 0 degrees
- moved D34 0.51 mm to (117.4, 41.0)
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Routing:
- net Net-(D34-Pad2): track 8.74 -> 0.00 mm
- net +5V: track 150.7 -> 145.4 mm
- net GND: track 158.2 -> 162.0 mm
- net Net-(JP2-Pad2): track 17.1 -> 19.0 mm
- net Net-(JP1-Pad2): track 11.6 -> 12.8 mm
- net Net-(R6-Pad1): track 2.67 -> 3.81 mm
- net Net-(C4-Pad1): track 5.37 -> 4.28 mm
- net Net-(R3-Pad1): track 1.53 -> 2.40 mm
- net Net-(R1-Pad2): track 5.19 -> 5.98 mm
- net Net-(Cx1-Pad1): track 41.3 -> 41.8 mm

Commit message: Add files via upload
Parts:
- D35: value TVS -> D_TVS_unidirection
- U1: value MT9284 -> MT9284_1
- moved D35 0.29 mm to (129.2, 43.8), turned to -90 degrees
Connections:
- D35 pad 1: GND -> +5V
- D35 pad 2: +5V -> GND

Commit message: Add files via upload
Parts:
- L1: footprint Inductor_SMD:L_WHC_0630_custom -> custom_footprint_library:L_WHC_0630_custom
- Rx1: footprint Resistor_SMD:R_1206_3216Metric -> custom_footprint_library:R_1206_0805_3216Metric_custom
- moved L1 4.42 mm to (125.2, 42.7)
- moved D20 3.55 mm to (85.9, 48.3)
- moved D28 3.55 mm to (85.9, 52.7)
- moved U1 3.55 mm to (122.8, 47.6)
- moved H2 3.55 mm to (41.8, 46.9)
- moved D12 3.55 mm to (85.9, 44.0)
- moved D4 3.55 mm to (85.9, 39.6)
- moved R3 3.55 mm to (120.2, 51.2)
- moved C3 3.55 mm to (121.1, 51.2)
- moved Cx1 3.55 mm to (119.2, 48.4)
- moved D17 3.55 mm to (114.6, 48.3)
- moved D18 3.55 mm to (105.0, 48.3)
- moved D19 3.55 mm to (95.5, 48.3)
- moved D21 3.55 mm to (76.4, 48.3)
- moved D22 3.55 mm to (66.8, 48.3)
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Routing:
- net +5V: track 145.3 -> 149.2 mm
- net Net-(D16-Pad1): track 259.3 -> 260.0 mm
- net GND: track 161.7 -> 162.3 mm

Commit message: Add files via upload
Parts:
- moved D34 0.34 mm to (118.7, 44.1)
Changed lines of the file:
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@@
   )
   (footprint "Diode_SMD:D_SMA" (layer "F.Cu")
-    (at 118.99 44.125 90)
+    (at 118.65 44.125 90)
     (descr "Diode SMA (DO-214AC)")
     (tags "Diode SMA (DO-214AC)")
@@
   (segment (start 123.34 47.615) (end 123.9275 47.615) (width 0.3) (layer "F.Cu") (net 14))
   (segment (start 125.2 46.005) (end 122.93 46.005) (width 0.3) (layer "F.Cu") (net 14))
-  (segment (start 118.445 48.365) (end 118.445 46.67) (width 0.75) (layer "F.Cu") (net 14))
   (segment (start 125.2 43.185) (end 125.2 46.005) (width 0.3) (layer "F.Cu") (net 14))
+  (segment (start 118.445 48.365) (end 118.445 46.33) (width 0.75) (layer "F.Cu") (net 14))
   (segment (start 115.495 39.625) (end 115.495 44.025) (width 1.215) (layer "F.Cu") (net 14))
   (segment (start 115.495 46.22) (end 115.495 48.325) (width 1.215) (layer "F.Cu") (net 14))
+  (segment (start 118.445 46.33) (end 118.65 46.125) (width 0.75) (layer "F.Cu") (net 14))
   (segment (start 115.495 44.025) (end 115.495 46.22) (width 1.215) (layer "F.Cu") (net 14))
-  (segment (start 118.99 46.125) (end 115.59 46.125) (width 1.35) (layer "F.Cu") (net 14))
   (segment (start 122.76 46.175) (end 122.76 47.035) (width 0.3) (layer "F.Cu") (net 14))
   (segment (start 117.045 38.075) (end 115.495 39.625) (width 0.3) (layer "F.Cu") (net 14))
+  (segment (start 115.495 46.22) (end 115.59 46.125) (width 1.215) (layer "F.Cu") (net 14))
   (segment (start 122.76 47.035) (end 123.34 47.615) (width 0.3) (layer "F.Cu") (net 14))
-  (segment (start 115.59 46.125) (end 115.495 46.22) (width 0.25) (layer "F.Cu") (net 14))
   (segment (start 125.205 43.15) (end 125.205 38.782842) (width 0.3) (layer "F.Cu") (net 14))
   (segment (start 122.93 46.005) (end 122.76 46.175) (width 0.3) (layer "F.Cu") (net 14))
   (segment (start 124.461802 38.075) (end 117.045 38.075) (width 0.3) (layer "F.Cu") (net 14))
-  (segment (start 118.445 46.67) (end 118.99 46.125) (width 0.75) (layer "F.Cu") (net 14))
   (segment (start 115.495 48.325) (end 115.495 52.725) (width 1.215) (layer "F.Cu") (net 14))
+  (segment (start 115.59 46.125) (end 118.65 46.125) (width 1.215) (layer "F.Cu") (net 14))
   (arc (start 125.005 38.3) (mid 124.755779 38.133475) (end 124.461802 38.075) (width 0.3) (layer "F.Cu") (net 14))
   (arc (start 125.205 38.782842) (mid 125.153022 38.52153) (end 125.005 38.3) (width 0.3) (layer "F.Cu") (net 14))
@@
         (xy 120.27 46.835)
         (xy 120.260075 43.584697)
-        (xy 116.940938 43.584302)
-        (xy 116.950945 37.374625)
+        (xy 116.865938 43.584181)
+        (xy 116.875945 37.374504)
         (xy 124.655536 37.387039)
       )
