File: USB_LEDs_2835/USB_LEDs_2835.kicad_pcb (KiCad board)
At the start: 2 copper layers, 99.9 x 20 mm, 56 parts, among them U1 MT9284_1, U2 JL8022W-L, U3 74LVC1G04

Commit message: Add files via upload
Parts:
- moved D35 2.33 mm to (130.8, 49.2)
Routing:
- net +5V: track 149.2 -> 151.0 mm
- net GND: track 162.3 -> 160.8 mm
Changed lines of the file:
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@@
   )
   (footprint "Diode_SMD:D_SOD-923" (layer "F.Cu")
-    (at 130.755 46.925 -90)
+    (at 130.75 49.25 -90)
     (descr "https://www.onsemi.com/pub/Collateral/ESD9B-D.PDF#page=4")
     (tags "Diode SOD923")
@@
     (property "Sheetname" "")
     (attr smd)
-    (fp_text reference "D35" (at -1.1 0 180) (layer "F.SilkS")
+    (fp_text reference "D35" (at 0 0.8 -90) (layer "F.SilkS")
       (effects (font (size 0.3 0.3) (thickness 0.07)))
     )
@@
   (segment (start 39.68 54.7) (end 38.076015 54.7) (width 0.3) (layer "F.Cu") (net 2))
   (segment (start 39.68 54.7) (end 42.795 54.7) (width 0.3) (layer "F.Cu") (net 2))
+  (segment (start 130.75 49.67) (end 130.455 49.965) (width 0.25) (layer "F.Cu") (net 2))
   (segment (start 36.88 51.425) (end 36.78 51.525) (width 0.2) (layer "F.Cu") (net 2))
   (segment (start 42.795 54.7) (end 42.89 54.605) (width 0.3) (layer "F.Cu") (net 2))
@@
   (segment (start 119.225723 55.935) (end 44.177715 55.935) (width 0.3) (layer "F.Cu") (net 2))
   (segment (start 39.2 43.515) (end 39.2 42.475) (width 0.3) (layer "F.Cu") (net 2))
+  (segment (start 130.455 49.965) (end 126.84 49.965) (width 0.25) (layer "F.Cu") (net 2))
   (segment (start 122.32 47.615) (end 122.79 48.085) (width 0.4) (layer "F.Cu") (net 2))
   (segment (start 121.6525 47.615) (end 122.32 47.615) (width 0.4) (layer "F.Cu") (net 2))
-  (segment (start 128.697036 49.965) (end 126.84 49.965) (width 0.25) (layer "F.Cu") (net 2))
   (segment (start 43.73 48.075) (end 43.055 48.75) (width 0.25) (layer "F.Cu") (net 2))
   (segment (start 42.89 54.647285) (end 42.89 54.605) (width 0.3) (layer "F.Cu") (net 2))
@@
   (segment (start 124.50596 55.94904) (end 119.239763 55.94904) (width 0.3) (layer "F.Cu") (net 2))
   (segment (start 126.855 48.400978) (end 126.129022 47.675) (width 0.3) (layer "F.Cu") (net 2))
-  (segment (start 130.755 47.345) (end 130.755 47.362564) (width 0.25) (layer "F.Cu") (net 2))
   (segment (start 121.12 51.665) (end 121.2 51.585) (width 0.25) (layer "F.Cu") (net 2))
   (segment (start 37.71 43.255) (end 38.16 43.705) (width 0.3) (layer "F.Cu") (net 2))
   (arc (start 36.205 53.925) (mid 34.243713 50.989726) (end 33.555 47.527335) (width 0.3) (layer "F.Cu") (net 2))
-  (arc (start 130.755 47.362564) (mid 130.527595 48.505806) (end 129.88 49.475) (width 0.25) (layer "F.Cu") (net 2))
   (arc (start 39.72 54.603432) (mid 39.709604 54.655694) (end 39.68 54.7) (width 0.2) (layer "F.Cu") (net 2))
-  (arc (start 129.88 49.475) (mid 129.337251 49.837653) (end 128.697036 49.965) (width 0.25) (layer "F.Cu") (net 2))
   (arc (start 38.076015 54.7) (mid 37.063429 54.498584) (end 36.205 53.925) (width 0.3) (layer "F.Cu") (net 2))
   (segment (start 44.9 48.215) (end 44.37 48.215) (width 0.4) (layer "F.Cu") (net 3))
@@
   (segment (start 127.405 41.237102) (end 127.405 42.725) (width 0.4) (layer "F.Cu") (net 3))
   (segment (start 45.36048 37.52548) (end 124.477618 37.52548) (width 0.4) (layer "F.Cu") (net 3))
-  (segment (start 130.755 45.625) (end 130.175 45.045) (width 0.25) (layer "F.Cu") (net 3))
   (segment (start 119.429996 53.354996) (end 119.429996 52.645003) (width 0.25) (layer "F.Cu") (net 3))
+  (segment (start 129.395 45.045) (end 127.405 45.045) (width 0.25) (layer "F.Cu") (net 3))
   (segment (start 43.8 37.445) (end 45.28 37.445) (width 0.4) (layer "F.Cu") (net 3))
-  (segment (start 130.175 45.045) (end 127.405 45.045) (width 0.25) (layer "F.Cu") (net 3))
   (segment (start 117.17702 51.97702) (end 118.65 51.97702) (width 0.4) (layer "F.Cu") (net 3))
-  (segment (start 130.755 45.625) (end 130.755 46.505) (width 0.25) (layer "F.Cu") (net 3))
   (segment (start 42.575 38.67) (end 43.8 37.445) (width 0.4) (layer "F.Cu") (net 3))
   (segment (start 114.105 54.125) (end 114.105 37.43) (width 0.2) (layer "F.Cu") (net 3))
@@
   (segment (start 125.735 46.715) (end 127.405 45.045) (width 0.4) (layer "F.Cu") (net 3))
   (segment (start 122.24 53.835) (end 119.91 53.835) (width 0.25) (layer "F.Cu") (net 3))
+  (segment (start 130.75 46.4) (end 129.395 45.045) (width 0.25) (layer "F.Cu") (net 3))
   (segment (start 125.25 46.665) (end 125.3 46.715) (width 0.25) (layer "F.Cu") (net 3))
   (segment (start 45.12 48.435) (end 45.12 37.605) (width 0.4) (layer "F.Cu") (net 3))
   (segment (start 45.12 37.605) (end 45.28 37.445) (width 0.4) (layer "F.Cu") (net 3))
+  (segment (start 130.75 48.83) (end 130.75 46.4) (width 0.25) (layer "F.Cu") (net 3))
   (arc (start 126.155469 38.220468) (mid 127.080257 39.604511) (end 127.405 41.237102) (width 0.4) (layer "F.Cu") (net 3))
   (arc (start 124.477618 37.52548) (mid 125.385664 37.706102) (end 126.155469 38.220468) (width 0.4) (layer "F.Cu") (net 3))
@@
     )
   )
+  (zone (net 3) (net_name "+5V") (layer "F.Cu") (hatch edge 0.508)
+    (priority 1)
+    (connect_pads (clearance 0.4))
+    (min_thickness 0.254) (filled_areas_thickness no)
+    (fill yes (thermal_gap 0.508) (thermal_bridge_width 0.508))
+    (polygon
+      (pts
+        (xy 126.15 37.2)
+        (xy 126.95 37.5)
+        (xy 128 38)
+        (xy 129.25 38.9)
+        (xy 130.25 39.85)
+        (xy 131.25 41.2)
+        (xy 131.95 42.65)
+        (xy 132.4 44)
+        (xy 132.6 45.35)
+        (xy 132.5 49)
+        (xy 129.55 49)
+        (xy 128.4 47)
+        (xy 125 47)
+        (xy 125 46.4)
+        (xy 125.45 46.4)
+        (xy 125.75 45.9)
+        (xy 125.75 37.1)
+      )
+    )
+  )
   (zone (net 24) (net_name "Net-(D19-Pad1)") (layer "F.Cu") (hatch edge 0.508)
     (priority 4)
@@
     )
   )
-  (zone (net 3) (net_name "+5V") (layer "F.Cu") (hatch edge 0.508)
-    (priority 1)
-    (connect_pads (clearance 0.4))
-    (min_thickness 0.254) (filled_areas_thickness no)
-    (fill yes (thermal_gap 0.508) (thermal_bridge_width 0.508))
-    (polygon
-      (pts
-        (xy 126.15 37.225)
-        (xy 127.05 37.55)
-        (xy 128.025 38.05)
-        (xy 128.95 38.65)
-        (xy 129.725 39.3)
-        (xy 130.35 39.975)
-        (xy 130.9 40.65)
-        (xy 131.375 41.4)
-        (xy 131.8 42.225)
-        (xy 132.125 43.025)
-        (xy 132.35 43.9)
-        (xy 132.525 44.7)
-        (xy 132.575 45.425)
-        (xy 132.575 46.975)
-        (xy 124.55 46.975)
-        (xy 124.55 46.35)
-        (xy 125.75 45.95)
-        (xy 125.75 37.1)
-      )
-    )
-  )
   (zone (net 0) (net_name "") (layer "F.Mask") (hatch edge 0.508)
     (connect_pads (clearance 0.4))
@@
     (polygon
       (pts
-        (xy 126.475 37.325)
-        (xy 126.9 37.5)
-        (xy 127.425 37.75)
-        (xy 128 38.025)
-        (xy 128.9 38.625)
-        (xy 129.35 38.975)
-        (xy 129.85 39.425)
-        (xy 130.275 39.875)
-        (xy 130.7 40.4)
-        (xy 131.05 40.9)
-        (xy 131.375 41.425)
-        (xy 131.7 42.025)
-        (xy 131.975 42.625)
-        (xy 132.225 43.35)
-        (xy 132.375 44.025)
-        (xy 132.5 44.65)
-        (xy 132.575 45.4)
-        (xy 132.575 47.975)
-        (xy 132.55 48.675)
-        (xy 132.45 49.3)
-        (xy 132.3 49.975)
-        (xy 132.1 50.65)
-        (xy 131.875 51.225)
-        (xy 131.575 51.85)
-        (xy 131.25 52.425)
-        (xy 130.9 53)
-        (xy 130.55 53.45)
-        (xy 130.1 53.95)
-        (xy 129.625 54.425)
-        (xy 129.175 54.825)
-        (xy 128.725 55.15)
-        (xy 128.175 55.5)
-        (xy 127.65 55.8)
-        (xy 127 56.1)
-        (xy 127 48.15)
-        (xy 125.75 45.95)
+        (xy 126.35 37.3)
+        (xy 127.2 37.6)
+        (xy 128.45 38.3)
+        (xy 129.45 39.05)
+        (xy 130.3 39.9)
+        (xy 131.15 41.05)
+        (xy 131.75 42.1)
+        (xy 132.15 43.05)
+        (xy 132.4 44.15)
+        (xy 132.6 45.3)
+        (xy 132.6 47.3)
+        (xy 132.55 48.5)
+        (xy 132.4 49.6)
+        (xy 132.05 50.8)
+        (xy 131.5 52.05)
+        (xy 130.75 53.15)
+        (xy 129.85 54.2)
+        (xy 128.75 55.15)
+        (xy 127.35 55.95)
+        (xy 125.9 56.5)
+        (xy 124.5 56.75)
+        (xy 124.5 55.4)
+        (xy 125.35 54.6)
+        (xy 125.35 53.45)
+        (xy 127 51.8)
+        (xy 127 47.95)
+        (xy 125.75 46.15)
         (xy 125.75 37.1)
       )
