File: USB_LEDs_2835/USB_LEDs_2835.kicad_pcb (KiCad board)
At the start: 2 copper layers, 99.9 x 20 mm, 56 parts, among them U1 MT9284_1, U2 JL8022W-L, U3 74LVC1G04

Commit message: Add files via upload
Parts:
- moved L1 0.48 mm to (125.2, 42.2)
Changed lines of the file:
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@@
+    )
+  )
+  (footprint "custom_footprint_library:L_WHC_0630_custom" (layer "F.Cu")
+    (at 125.2 42.25 180)
+    (descr "smd shielded power inductor http://www.abracon.com/Magnetics/power/ASPI-3012S.pdf")
+    (tags "inductor abracon smd shielded")
+    (property "Sheetfile" "USB_LEDs_2835.kicad_sch")
+    (property "Sheetname" "")
+    (zone_connect 2)
+    (attr smd)
+    (fp_text reference "L1" (at -0.01 2.91) (layer "F.SilkS")
+      (effects (font (size 0.5 0.5) (thickness 0.1)))
+    )
+    (fp_text value "L_Ferrite_Small" (at 0 3.29) (layer "F.Fab") hide
+      (effects (font (size 1 1) (thickness 0.15)))
+    )
+    (fp_text user "${REFERENCE}" (at 0.025 -1.36) (layer "F.Fab") hide
+      (effects (font (size 0.7 0.7) (thickness 0.105)))
+    )
+    (fp_line (start -0.775 2.35) (end 0.825 2.35) (layer "F.SilkS") (width 0.12))
+    (fp_line (start -0.775 -2.35) (end 0.825 -2.35) (layer "F.SilkS") (width 0.12))
+    (fp_line (start 4.15 -2.45) (end -4.15 -2.45) (layer "F.CrtYd") (width 0.05))
+    (fp_line (start 4.15 2.45) (end 4.15 -2.45) (layer "F.CrtYd") (width 0.05))
+    (fp_line (start -4.15 -2.45) (end -4.15 2.45) (layer "F.CrtYd") (width 0.05))
+    (fp_line (start -4.15 2.45) (end 4.15 2.45) (layer "F.CrtYd") (width 0.05))
+    (fp_line (start 3.0775 2.05) (end 3.08 -2.05) (layer "F.Fab") (width 0.1))
+    (fp_line (start -0.975 -2.05) (end -3.09 -2.05) (layer "F.Fab") (width 0.1))
+    (fp_line (start -0.975 2.05) (end -0.775 2.25) (layer "F.Fab") (width 0.1))
+    (fp_line (start 0.825 -2.25) (end -0.775 -2.25) (layer "F.Fab") (width 0.1))
+    (fp_line (start 3.08 -2.05) (end 1.025 -2.05) (layer "F.Fab") (width 0.1))
+    (fp_line (start -3.09 2.05) (end -0.975 2.05) (layer "F.Fab") (width 0.1))
+    (fp_line (start -0.775 2.25) (end 0.825 2.25) (layer "F.Fab") (width 0.1))
+    (fp_line (start 0.825 2.25) (end 1.025 2.05) (layer "F.Fab") (width 0.1))
+    (fp_line (start 1.025 -2.05) (end 0.825 -2.25) (layer "F.Fab") (width 0.1))
+    (fp_line (start -3.09 -2.05) (end -3.09 2.05) (layer "F.Fab") (width 0.1))
+    (fp_line (start -0.775 -2.25) (end -0.975 -2.05) (layer "F.Fab") (width 0.1))
+    (fp_line (start 1.0225 2.05) (end 3.0775 2.05) (layer "F.Fab") (width 0.1))
+    (pad "1" smd rect (at -2.3 0 180) (size 3.1 3.5) (layers "F.Cu" "F.Paste" "F.Mask")
+      (net 3 "+5V") (pintype "passive") (zone_connect 2))
+    (pad "2" smd rect (at 2.3 0 180) (size 3.1 3.5) (layers "F.Cu" "F.Paste" "F.Mask")
+      (net 36 "Net-(D34-Pad2)") (pintype "passive") (zone_connect 2))
+    (model "${KICAD6_3DMODEL_DIR}/Inductor_SMD.3dshapes/L_Abracon_ASPI-3012S.wrl"
+      (offset (xyz 0 0 0))
+      (scale (xyz 1 1 1))
+      (rotate (xyz 0 0 0))
     )
   )
@@
       (offset (xyz 0 0 0))
       (scale (xyz 1 1 1))
-      (rotate (xyz 0 0 0))
-    )
-  )
-  (footprint "custom_footprint_library:L_WHC_0630_custom" (layer "F.Cu")
-    (at 125.205 42.725 180)
-    (descr "smd shielded power inductor http://www.abracon.com/Magnetics/power/ASPI-3012S.pdf")
-    (tags "inductor abracon smd shielded")
-    (property "Sheetfile" "USB_LEDs_2835.kicad_sch")
-    (property "Sheetname" "")
-    (zone_connect 2)
-    (attr smd)
-    (fp_text reference "L1" (at -0.045 3.025) (layer "F.SilkS")
-      (effects (font (size 0.5 0.5) (thickness 0.1)))
-    )
-    (fp_text value "L_Ferrite_Small" (at 0 3.29) (layer "F.Fab") hide
-      (effects (font (size 1 1) (thickness 0.15)))
-    )
-    (fp_text user "${REFERENCE}" (at 0.025 -1.36) (layer "F.Fab")
-      (effects (font (size 0.7 0.7) (thickness 0.105)))
-    )
-    (fp_line (start -0.775 -2.35) (end 0.825 -2.35) (layer "F.SilkS") (width 0.12))
-    (fp_line (start -0.775 2.55) (end 0.825 2.55) (layer "F.SilkS") (width 0.12))
-    (fp_line (start -4.15 2.65) (end 4.15 2.65) (layer "F.CrtYd") (width 0.05))
-    (fp_line (start 4.15 -2.45) (end -4.15 -2.45) (layer "F.CrtYd") (width 0.05))
-    (fp_line (start -4.15 -2.45) (end -4.15 2.65) (layer "F.CrtYd") (width 0.05))
-    (fp_line (start 4.15 2.65) (end 4.15 -2.45) (layer "F.CrtYd") (width 0.05))
-    (fp_line (start 0.825 2.45) (end 1.025 2.25) (layer "F.Fab") (width 0.1))
-    (fp_line (start -0.775 2.45) (end 0.825 2.45) (layer "F.Fab") (width 0.1))
-    (fp_line (start -0.775 -2.25) (end -0.975 -2.05) (layer "F.Fab") (width 0.1))
-    (fp_line (start -3.09 2.25) (end -0.975 2.25) (layer "F.Fab") (width 0.1))
-    (fp_line (start 3.08 -2.05) (end 1.025 -2.05) (layer "F.Fab") (width 0.1))
-    (fp_line (start 1.025 -2.05) (end 0.825 -2.25) (layer "F.Fab") (width 0.1))
-    (fp_line (start -3.09 -2.05) (end -3.09 2.25) (layer "F.Fab") (width 0.1))
-    (fp_line (start 1.025 2.25) (end 3.08 2.25) (layer "F.Fab") (width 0.1))
-    (fp_line (start 0.825 -2.25) (end -0.775 -2.25) (layer "F.Fab") (width 0.1))
-    (fp_line (start -0.975 -2.05) (end -3.09 -2.05) (layer "F.Fab") (width 0.1))
-    (fp_line (start 3.08 2.25) (end 3.08 -2.05) (layer "F.Fab") (width 0.1))
-    (fp_line (start -0.975 2.25) (end -0.775 2.45) (layer "F.Fab") (width 0.1))
-    (pad "1" smd rect (at -2.2 0 180) (size 3.3 3.5) (layers "F.Cu" "F.Paste" "F.Mask")
-      (net 3 "+5V") (pintype "passive") (zone_connect 2))
-    (pad "2" smd rect (at 2.2 0 180) (size 3.3 3.5) (layers "F.Cu" "F.Paste" "F.Mask")
-      (net 36 "Net-(D34-Pad2)") (pintype "passive") (zone_connect 2))
-    (model "${KICAD6_3DMODEL_DIR}/Inductor_SMD.3dshapes/L_Abracon_ASPI-3012S.wrl"
-      (offset (xyz 0 0 0))
-      (scale (xyz 1 1 1))

Commit message: Add files via upload
Parts:
- moved Cx1 4.68 mm to (120.8, 52.8)
- moved L1 3.64 mm to (121.8, 40.9)
- moved D34 3.58 mm to (118.7, 47.7)
- moved R1 2.79 mm to (123.2, 53.4)
- moved U3 2.45 mm to (125.6, 52.7)
- moved Rx1 1.53 mm to (118.1, 53.5)
- moved C2 1.51 mm to (125.2, 45.7)
- moved C3 1.48 mm to (122.1, 50.1)
- moved R2 1.48 mm to (121.7, 48.7)
- moved R3 1.48 mm to (121.2, 50.1)
- moved D33 1.42 mm to (125.7, 48.4)
- moved U1 1.22 mm to (122.7, 46.4)
- moved R4 0.51 mm to (123.7, 50.5)
- moved C4 0.51 mm to (123.7, 49.6)
Routing:
- net GND: track 160.8 -> 173.9 mm
- net Net-(D34-Pad2): track 0.00 -> 8.18 mm
- net Net-(Cx1-Pad1): track 41.3 -> 37.3 mm
- net Net-(D33-Pad2): track 94.2 -> 97.1 mm
- net Net-(D16-Pad1): track 260.0 -> 262.1 mm
- net Net-(R3-Pad1): track 2.40 -> 4.25 mm
- net Net-(R1-Pad2): track 5.92 -> 7.61 mm
- net +5V: track 151.0 -> 149.7 mm
- net Net-(C4-Pad1): track 4.28 -> 5.24 mm
- net Net-(JP2-Pad2): track 19.0 -> 18.2 mm
Other:
- board text added: "JLCJLCJLCJLC"

Commit message: Add files via upload
Parts:
- moved L1 0.27 mm to (121.8, 40.6)
- moved D34 0.25 mm to (118.7, 47.5)
- moved Rx1 0.23 mm to (118.1, 53.3)

Commit message: Add files via upload
Parts:
- C2: footprint Capacitor_SMD:C_0402_1005Metric -> Capacitor_SMD:C_0603_1608Metric
- moved D33 0.49 mm to (125.7, 48.9)
- moved C2 0.31 mm to (125.5, 45.6)
Routing:
- net GND: track 173.9 -> 172.9 mm
- net Net-(D33-Pad2): track 96.8 -> 96.2 mm
Other:
- board text removed: "JLCJLCJLCJLC"
