File: USB_LEDs_2835/panel/panel.kicad_pcb (KiCad board)
At the start: 2 copper layers, 105.9 x 100 mm, 280 parts, among them U1 MT9284_1, U2 JL8022W-L, U3 74LVC1G04

Commit message: Add files via upload
Other:
- board size 105.9 x 100 mm -> 99.9 x 100 mm
- board text removed: "JLCJLCJLCJLC"

Commit message: Add files via upload
Other:
- board text added: "JLCJLCJLCJLC"

Commit message: Add files via upload
Other:
- board size 99.9 x 100 mm -> 105.9 x 100 mm
- board text removed: "JLCJLCJLCJLC"
